File: electronics/bike_CVT_test_jig_V000/bike_CVT_test_jig_V000.kicad_pcb (KiCad board)
At the start: 2 copper layers, 90 x 98 mm, 42 parts, among them J13 Conn_01x03, J14 Conn_01x03, J15 Conn_01x03, J16 Conn_01x03, J17 Conn_01x03, J18 Conn_01x03, J19 Conn_01x03, J20 Conn_01x03, J21 Conn_01x03, J22 Conn_01x03, J23 Conn_01x03, J24 Conn_01x03, SW1 switch_DPDT, SW2 switch_DPDT, SW3 switch_DPDT, SW4 switch_DPDT

Commit message: added power connectors
Parts:
- removed C2, C3, C4: 10n, SquantorRcl:C_0805+0603
- removed J13, J14, J15, J16, J17, J18, J20, J21, J22, J23, J24: Conn_01x03, Connector_JST:JST_PH_B3B-PH-K_1x03_P2.00mm_Vertical
- removed LED1, LED3, LED4: LED_Dual_CC, SquantorDiodes:LED_DUAL_TH245_90deg
- removed R10, R11, R12, R5, R6, R9: R, SquantorRcl:R_0603_hand
- removed R2, R3, R4: 1K, SquantorRcl:R_0805+0603
- removed SW1, SW2, SW3, SW4: switch_DPDT, SquantorSwitches:PS-22F02
- added F1: Fuse, Fuse:Fuse_BelFuse_0ZRE0033FF_L11.4mm_W3.8mm, F.Cu at (119.5, 63.6)
- added F2: Fuse, Fuse:Fuse_BelFuse_0ZRE0033FF_L11.4mm_W3.8mm, F.Cu at (115.2, 63.6)
- added J1: Conn_02x02_Counter_Clockwise, Connector_Molex:Molex_Mini-Fit_Jr_5566-04A_2x02_P4.20mm_Vertical, F.Cu at (121.4, 52.2)
- C1, R1: moved to F.Cu
- moved C1 9.65 mm to (134.3, 49.8)
- moved R1 9.65 mm to (134.3, 46.5)
- moved J19 9.50 mm to (196.6, 129.6)
- moved R7 9.50 mm to (196.6, 131.5)
- moved R8 9.50 mm to (201.0, 131.5)
- moved LED2 1.31 mm to (198.7, 134.5)
Connections:
- H2 pad 1: Net-(C2-Pad1) -> (no net)
- H3 pad 1: Net-(C3-Pad1) -> (no net)
- H4 pad 1: Net-(C4-Pad1) -> (no net)
Routing:
- net Net-(J15-Pin_3): track 17.3 -> 0.00 mm
- net Net-(J18-Pin_1): track 17.1 -> 0.00 mm
- net Net-(J16-Pin_3): track 16.2 -> 0.00 mm
- net Net-(J23-Pin_1): track 16.1 -> 0.00 mm
- net Net-(J24-Pin_3): track 13.8 -> 0.00 mm
- net Net-(J13-Pin_1): track 13.8 -> 0.00 mm
- net Net-(J18-Pin_2): track 13.3 -> 0.00 mm
- net Net-(J15-Pin_2): track 12.9 -> 0.00 mm
- net Net-(J16-Pin_2): track 12.9 -> 0.00 mm
- net Net-(J23-Pin_2): track 12.8 -> 0.00 mm
- net Net-(J14-Pin_2): track 12.5 -> 0.00 mm
- net Net-(J22-Pin_1): track 12.4 -> 0.00 mm
- net Net-(J17-Pin_3): track 12.0 -> 0.00 mm
- net Net-(J21-Pin_2): track 11.8 -> 0.00 mm
- net Net-(J20-Pin_2): track 11.8 -> 0.00 mm
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