File: electronics/bike_CVT_test_jig_V000/bike_CVT_test_jig_V000.kicad_sch (KiCad schematic)
At the start: 42 parts, among them J13 Conn_01x03, J14 Conn_01x03, J15 Conn_01x03, J16 Conn_01x03, J17 Conn_01x03, J18 Conn_01x03, J19 Conn_01x03, J20 Conn_01x03, J21 Conn_01x03, J22 Conn_01x03, J23 Conn_01x03, J24 Conn_01x03, SW1 switch_DPDT, SW2 switch_DPDT, SW3 switch_DPDT, SW4 switch_DPDT

Commit message: added power connectors
Parts:
- removed C2, C3, C4: 10n, SquantorRcl:C_0805+0603, symbol Device:C
- removed J13, J14, J15, J16, J17, J18, J20, J21, J22, J23, J24: Conn_01x03, Connector_JST:JST_PH_B3B-PH-K_1x03_P2.00mm_Vertical, symbol Connector_Generic:Conn_01x03
- removed LED1, LED3, LED4: LED_Dual_CC, SquantorDiodes:LED_DUAL_TH245_90deg, symbol SquantorDevice:LED_Dual_CC
- removed R10, R11, R12, R5, R6, R9: R, SquantorRcl:R_0603_hand, symbol Device:R
- removed R2, R3, R4: 1K, SquantorRcl:R_0805+0603, symbol Device:R
- removed SW1, SW2, SW3, SW4: switch_DPDT, SquantorSwitches:PS-22F02, symbol SquantorSwitches:switch_DPDT
- added F1, F2: Fuse, Fuse:Fuse_BelFuse_0ZRE0033FF_L11.4mm_W3.8mm, symbol Device:Fuse
- added J1: Conn_02x02_Counter_Clockwise, Connector_Molex:Molex_Mini-Fit_Jr_5566-04A_2x02_P4.20mm_Vertical, symbol Connector_Generic:Conn_02x02_Counter_Clockwise
- H2, H3, H4: symbol Mechanical:MountingHole_Pad -> Mechanical:MountingHole
Connections:
- net GND: now also J1.3 (Pin_3), J1.4 (Pin_4); no longer C1.2, R1.2
- new net: F1.2, J1.1 (Pin_1)
- new net: F2.2, J1.2 (Pin_2)
- new net: C1.2, R1.2
- new net +24V: F1.1
- new net +5V: F2.1
Other:
- added sheet stepstick (stepstick.kicad_sch)

Commit message: schematic entry work in progress
Connections:
- net GND: now also C1.2, R1.2
Changed lines of the file:
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@@
   (junction (at 152.4 168.91) (diameter 0) (color 0 0 0 0)
+  )
+  (junction (at 152.4 165.1) (diameter 0) (color 0 0 0 0)
   )
   (wire (pts (xy 22.86 24.13) (xy 24.13 24.13))
@@
     (stroke (width 0) (type default))
   )
+  (wire (pts (xy 152.4 165.1) (xy 153.67 165.1))
+    (stroke (width 0) (type default))
+  )
